Commit message: Updating changes

File: src/my_robo1_py_pkg/urdf/my_robo1.urdf.xacro (robot description, xacro)
@@ -45,5 +45,5 @@
         <cylinder radius="${wheel_radius}" length="${wheel_width}"/>
       </geometry>
-      <material name="blue">
+      <material name="white">
         <color rgba="1 1 1 1"/>
       </material>
